Commit message: Times 10 all xacro parameters

File: gyro_description/urdf/component_snippets.xacro (robot description, xacro)
@@ -4,71 +4,67 @@
     <xacro:property name="PI" value="3.1415926535897931"/>
     <!-- Macro to add an IMU. -->
-  <xacro:macro name="imu_plugin_macro"
-    params="namespace imu_suffix parent_link imu_topic
+    <xacro:macro name="imu_plugin_macro"
+                 params="namespace imu_suffix parent_link imu_topic
       mass_imu_sensor gyroscope_noise_density gyroscope_random_walk
       gyroscope_bias_correlation_time gyroscope_turn_on_bias_sigma
       accelerometer_noise_density accelerometer_random_walk
-      accelerometer_bias_correlation_time accelerometer_turn_on_bias_sigma
+      accel_bias_correlation_time accelerometer_turn_on_bias_sigma
       *inertia *origin">
-    <!-- IMU link -->
-    <link name="${namespace}/imu${imu_suffix}_link">
-      <inertial>
-        <xacro:insert_block name="inertia" />
-        <mass value="${mass_imu_sensor}" />  <!-- [kg] -->
-        <origin xyz="0 0 0" rpy="0 0 0" />
-      </inertial>
-    </link>
-    <!-- IMU joint -->
-    <joint name="${namespace}/imu${imu_suffix}_joint" type="revolute">
-      <xacro:insert_block name="origin" />
-      <parent link="${parent_link}" />
-      <child link="${namespace}/imu${imu_suffix}_link" />
-      <limit upper="0" lower="0" effort="0" velocity="0" />
-    </joint>
-    <gazebo reference="imu_link">
-    <gravity>true</gravity>
-    <sensor name="imu_sensor" type="imu">
-      <always_on>true</always_on>
-      <update_rate>100</update_rate>
-      <visualize>true</visualize>
-      <plugin filename="libgazebo_ros_imu_sensor.so" name="imu_plugin">
-        <topicName>${imu_topic}</topicName>
-        <bodyName>imu_link</bodyName>
-        <updateRateHZ>10.0</updateRateHZ>
-        <gaussianNoise>0.0</gaussianNoise>
-        <xyzOffset>0 0 0</xyzOffset>
-        <rpyOffset>0 0 0</rpyOffset>
-        <frameName>imu_link</frameName>
-      </plugin>
-      <pose>0 0 0 0 0 0</pose>
-    </sensor>
-  </gazebo>
-    <gazebo>
-    <sensor name="imu_sensor" type="imu">
-        <always_on>true</always_on>
-        <update_rate>100</update_rate>
-        <visualize>true</visualize>
-        <topic>${imu_topic}</topic>
-      <plugin filename="libgazebo_ros_imu_sensor.so" name="imu_plugin">
-      <!-- A good description of the IMU parameters can be found in the kalibr documentation:
-           https://github.com/ethz-asl/kalibr/wiki/IMU-Noise-Model-and-Intrinsics -->
-        <robotNamespace>${namespace}</robotNamespace> <!-- (string, required): ros namespace in which the messages are published -->
-        <linkName>${namespace}/imu${imu_suffix}_link</linkName> <!-- (string, required): name of the body which holds the IMU sensor -->
-        <imuTopic>${imu_topic}</imuTopic> <!-- (string): name of the sensor output topic and prefix of service names (defaults to imu) -->
-        <gyroscopeNoiseDensity>${gyroscope_noise_density}</gyroscopeNoiseDensity> <!-- Gyroscope noise density (two-sided spectrum) [rad/s/sqrt(Hz)] -->
-        <gyroscopeRandomWalk>${gyroscope_random_walk}</gyroscopeRandomWalk> <!-- Gyroscope bias random walk [rad/s/s/sqrt(Hz)] -->
-        <gyroscopeBiasCorrelationTime>${gyroscope_bias_correlation_time}</gyroscopeBiasCorrelationTime> <!-- Gyroscope bias correlation time constant [s] -->
-        <gyroscopeTurnOnBiasSigma>${gyroscope_turn_on_bias_sigma}</gyroscopeTurnOnBiasSigma> <!-- Gyroscope turn on bias standard deviation [rad/s] -->
-        <accelerometerNoiseDensity>${accelerometer_noise_density}</accelerometerNoiseDensity> <!-- Accelerometer noise density (two-sided spectrum) [m/s^2/sqrt(Hz)] -->
-        <accelerometerRandomWalk>${accelerometer_random_walk}</accelerometerRandomWalk> <!-- Accelerometer bias random walk. [m/s^2/s/sqrt(Hz)] -->
-        <accelerometerBiasCorrelationTime>${accelerometer_bias_correlation_time}</accelerometerBiasCorrelationTime> <!-- Accelerometer bias correlation time constant [s] -->
-        <accelerometerTurnOnBiasSigma>${accelerometer_turn_on_bias_sigma}</accelerometerTurnOnBiasSigma> <!-- Accelerometer turn on bias standard deviation [m/s^2] -->
-      </plugin>
-      </sensor>
-    </gazebo>
-  </xacro:macro>
-   <!-- Macro to add a generic odometry sensor. -->
-  <xacro:macro name="odometry_plugin_macro"
-    params="
+        <!-- IMU link -->
+        <link name="${namespace}/imu${imu_suffix}_link">
+            <inertial>
+                <xacro:insert_block name="inertia"/>
+                <mass value="${mass_imu_sensor}"/>  <!-- [kg] -->
+                <origin xyz="0 0 0" rpy="0 0 0"/>
+            </inertial>
+        </link>
+        <!-- IMU joint -->
+        <joint name="${namespace}/imu${imu_suffix}_joint" type="fixed">
+            <xacro:insert_block name="origin"/>
+            <parent link="${parent_link}"/>
+            <child link="${namespace}/imu${imu_suffix}_link"/>
+<!--            <limit upper="0" lower="0" effort="0" velocity="0"/>-->
+        </joint>
+        <gazebo reference="${namespace}/imu${imu_suffix}_link">
+            <sensor name="imu_sensor" type="imu">
+                <always_on>true</always_on>
+                <update_rate>100</update_rate>
+                <visualize>true</visualize>
+                <plugin filename="libgazebo_ros_imu_sensor.so" name="imu_plugin">
+                    <!-- A good description of the IMU parameters can be found in the kalibr documentation:
+                         https://github.com/ethz-asl/kalibr/wiki/IMU-Noise-Model-and-Intrinsics -->
+                    <!-- (string, required): ros namespace in which the messages are published -->
+                    <robotNamespace>${namespace}</robotNamespace>
+                    <frameName>${namespace}/imu${imu_suffix}_link</frameName>
+                    <topicName>${imu_topic}</topicName>
+                    <updateRateHZ>10.0</updateRateHZ>
+                    <gaussianNoise>0.0</gaussianNoise>
+                    <xyzOffset>0 0 0</xyzOffset>
+                    <rpyOffset>0 0 0</rpyOffset>
+                    <!-- (string, required): name of the body which holds the IMU sensor -->
+                    <linkName>${namespace}/imu${imu_suffix}_link</linkName>
+                    <!-- Gyroscope noise density (two-sided spectrum) [rad/s/sqrt(Hz)] -->
+                    <gyroscopeNoiseDensity>${gyroscope_noise_density}</gyroscopeNoiseDensity>
+                    <!-- Gyroscope bias random walk [rad/s/s/sqrt(Hz)] -->
+                    <gyroscopeRandomWalk>${gyroscope_random_walk}</gyroscopeRandomWalk>
+                    <!-- Gyroscope bias correlation time constant [s] -->
+                    <gyroscopeBiasCorrelationTime>${gyroscope_bias_correlation_time}</gyroscopeBiasCorrelationTime>
+                    <!-- Gyroscope turn on bias standard deviation [rad/s] -->
+                    <gyroscopeTurnOnBiasSigma>${gyroscope_turn_on_bias_sigma}</gyroscopeTurnOnBiasSigma>
+                    <!-- Accelerometer noise density (two-sided spectrum) [m/s^2/sqrt(Hz)] -->
+                    <accelerometerNoiseDensity>${accelerometer_noise_density}</accelerometerNoiseDensity>
+                    <!-- Accelerometer bias random walk. [m/s^2/s/sqrt(Hz)] -->
+                    <accelerometerRandomWalk>${accelerometer_random_walk}</accelerometerRandomWalk>
+                    <!-- Accelerometer bias correlation time constant [s] -->
+                    <accelerometerBiasCorrelationTime>${accel_bias_correlation_time}</accelerometerBiasCorrelationTime>
+                    <!-- Accelerometer turn on bias standard deviation [m/s^2] -->
+                    <accelerometerTurnOnBiasSigma>${accelerometer_turn_on_bias_sigma}</accelerometerTurnOnBiasSigma>
+                </plugin>
+            </sensor>
+        </gazebo>
+    </xacro:macro>
+    <!-- Macro to add a generic odometry sensor. -->
+    <xacro:macro name="odometry_plugin_macro"
+                 params="
       namespace odometry_sensor_suffix parent_link pose_topic pose_with_covariance_topic
       position_topic transform_topic odometry_topic parent_frame_id child_frame_id
@@ -79,190 +75,225 @@
       noise_uniform_angular_velocity enable_odometry_map odometry_map
       image_scale *inertia *origin">
-    <!-- odometry link -->
-    <link name="${namespace}/odometry_sensor${odometry_sensor_suffix}_link">
-      <inertial>
-        <xacro:insert_block name="inertia" />
-        <mass value="${mass_odometry_sensor}" />  <!-- [kg] -->
-      </inertial>
-    </link>
-    <!-- odometry joint -->
-    <joint name="${namespace}/odometry_sensor${odometry_sensor_suffix}_joint" type="revolute">
-      <parent link="${parent_link}" />
-      <xacro:insert_block name="origin" />
-      <child link="${namespace}/odometry_sensor${odometry_sensor_suffix}_link" />
-      <limit upper="0" lower="0" effort="0" velocity="0" />
-    </joint>
-    <gazebo>
-      <plugin filename="librotors_gazebo_odometry_plugin.so" name="odometry_sensor${odometry_sensor_suffix}">
-        <linkName>${namespace}/odometry_sensor${odometry_sensor_suffix}_link</linkName>
-        <robotNamespace>${namespace}</robotNamespace>
-        <poseTopic>${pose_topic}</poseTopic>
-        <poseWithCovarianceTopic>${pose_with_covariance_topic}</poseWithCovarianceTopic>
-        <positionTopic>${position_topic}</positionTopic>
-        <transformTopic>${transform_topic}</transformTopic>
-        <odometryTopic>${odometry_topic}</odometryTopic>
-        <parentFrameId>${parent_frame_id}</parentFrameId> <!-- Use the scoped link name here. e.g. Model::link. -->
-        <childFrameId>${child_frame_id}</childFrameId>
-        <measurementDivisor>${measurement_divisor}</measurementDivisor> <!-- only every (seq % measurementDivisor) == 0 measurement is published [int] -->
-        <measurementDelay>${measurement_delay}</measurementDelay> <!-- time that measurement gets held back before it's published in [simulation cycles (int)] -->
-        <unknownDelay>${unknown_delay}</unknownDelay> <!-- additional delay, that just gets added to the timestamp [s] -->
-        <noiseNormalPosition>${noise_normal_position}</noiseNormalPosition> <!-- standard deviation of additive white gaussian noise [m] -->
-        <noiseNormalQuaternion>${noise_normal_quaternion}</noiseNormalQuaternion> <!-- standard deviation white gaussian noise [rad]: q_m = q*quaternionFromSmallAngleApproximation(noiseNormalQ) -->
-        <noiseNormalLinearVelocity>${noise_normal_linear_velocity}</noiseNormalLinearVelocity> <!-- standard deviation of additive white gaussian noise [m/s] -->
-        <noiseNormalAngularVelocity>${noise_normal_angular_velocity}</noiseNormalAngularVelocity> <!-- standard deviation of additive white gaussian noise [rad/s] -->
-        <noiseUniformPosition>${noise_uniform_position}</noiseUniformPosition> <!-- symmetric bounds of uniform noise [m] -->
-        <noiseUniformQuaternion>${noise_uniform_quaternion}</noiseUniformQuaternion> <!-- symmetric bounds of uniform noise [rad], computation see above -->
-        <noiseUniformLinearVelocity>${noise_uniform_linear_velocity}</noiseUniformLinearVelocity> <!-- symmetric bounds of uniform noise [m/s] -->
-        <noiseUniformAngularVelocity>${noise_uniform_angular_velocity}</noiseUniformAngularVelocity> <!-- symmetric bounds of uniform noise [rad/s] -->
-        <xacro:if value="${enable_odometry_map}">
-          <covarianceImage>package://vant3d_gazebo/resource/${odometry_map}</covarianceImage> <!-- a bitmap image describing where the sensor works (white), and where not (black) -->
-          <covarianceImageScale>${image_scale}</covarianceImageScale> <!-- the scale of the image in the gazebo world, if set to 1.0, 1 pixel in the image corresponds to 1 meter in the world -->
-        </xacro:if>
-      </plugin>
-    </gazebo>
-  </xacro:macro>
-  <!-- Macro to add a GPS sensor. -->
-  <xacro:macro name="gps_plugin_macro"
-    params="namespace gps_suffix parent_link gps_topic ground_speed_topic
+        <!-- odometry link -->
+        <link name="${namespace}/odometry_sensor${odometry_sensor_suffix}_link">
+            <inertial>
+                <xacro:insert_block name="inertia"/>
+                <mass value="${mass_odometry_sensor}"/>  <!-- [kg] -->
+            </inertial>
+        </link>
+        <!-- odometry joint -->
+        <joint name="${namespace}/odometry_sensor${odometry_sensor_suffix}_joint" type="revolute">
+            <parent link="${parent_link}"/>
+            <xacro:insert_block name="origin"/>
+            <child link="${namespace}/odometry_sensor${odometry_sensor_suffix}_link"/>
+            <limit upper="0" lower="0" effort="0" velocity="0"/>
+        </joint>
+        <gazebo>
+            <plugin filename="librotors_gazebo_odometry_plugin.so" name="odometry_sensor${odometry_sensor_suffix}">
+                <linkName>${namespace}/odometry_sensor${odometry_sensor_suffix}_link</linkName>
+                <robotNamespace>${namespace}</robotNamespace>
+                <poseTopic>${pose_topic}</poseTopic>
+                <poseWithCovarianceTopic>${pose_with_covariance_topic}</poseWithCovarianceTopic>
+                <positionTopic>${position_topic}</positionTopic>
+                <transformTopic>${transform_topic}</transformTopic>
+                <odometryTopic>${odometry_topic}</odometryTopic>
+                <!-- Use the scoped link name here. e.g. Model::link. -->
+                <parentFrameId>${parent_frame_id}</parentFrameId>
+                <childFrameId>${child_frame_id}</childFrameId>
+                <!-- only every (seq % measurementDivisor) == 0 measurement is published [int] -->
+                <measurementDivisor>${measurement_divisor}</measurementDivisor>
+                <!-- time that measurement gets held back before it's published in [simulation cycles (int)] -->
+                <measurementDelay>${measurement_delay}</measurementDelay>
+                <!-- additional delay, that just gets added to the timestamp [s] -->
+                <unknownDelay>${unknown_delay}</unknownDelay>
+                <!-- standard deviation of additive white gaussian noise [m] -->
+                <noiseNormalPosition>${noise_normal_position}</noiseNormalPosition>
+                <!-- standard deviation white gaussian noise
+                [rad]: q_m = q*quaternionFromSmallAngleApproximation(noiseNormalQ) -->
+                <noiseNormalQuaternion>${noise_normal_quaternion}</noiseNormalQuaternion>
+                <!-- standard deviation of additive white gaussian noise [m/s] -->
+                <noiseNormalLinearVelocity>${noise_normal_linear_velocity}</noiseNormalLinearVelocity>
+                <!-- standard deviation of additive white gaussian noise [rad/s] -->
+                <noiseNormalAngularVelocity>${noise_normal_angular_velocity}</noiseNormalAngularVelocity>
+                <!-- symmetric bounds of uniform noise [m] -->
+                <noiseUniformPosition>${noise_uniform_position}</noiseUniformPosition>
+                <!-- symmetric bounds of uniform noise [rad], computation see above -->
+                <noiseUniformQuaternion>${noise_uniform_quaternion}</noiseUniformQuaternion>
+                <!-- symmetric bounds of uniform noise [m/s] -->
+                <noiseUniformLinearVelocity>${noise_uniform_linear_velocity}</noiseUniformLinearVelocity>
+                <!-- symmetric bounds of uniform noise [rad/s] -->
+                <noiseUniformAngularVelocity>${noise_uniform_angular_velocity}</noiseUniformAngularVelocity>
+                <xacro:if value="${enable_odometry_map}">
+                    <!-- a bitmap image describing where the sensor works (white), and where not (black) -->
+                    <covarianceImageScale>${image_scale}
+                        <covarianceImage>package://vant3d_gazebo/resource/${odometry_map}</covarianceImage>
+                    </covarianceImageScale>
+                    <!-- the scale of the image in the gazebo world
+                     if set to 1.0, 1 pixel in the image corresponds to 1 meter in the world -->
+                </xacro:if>
+            </plugin>
+        </gazebo>
+    </xacro:macro>
+    <!-- Macro to add a GPS sensor. -->
+    <xacro:macro name="gps_plugin_macro"
+                 params="namespace gps_suffix parent_link gps_topic ground_speed_topic
       mass_gps_sensor horizontal_pos_std_dev vertical_pos_std_dev
       horizontal_vel_std_dev vertical_vel_std_dev *inertia *origin">
-    <!-- GPS link -->
-    <link name="${namespace}/gps${gps_suffix}_link">
-      <inertial>
-        <xacro:insert_block name="inertia" />
-        <mass value="${mass_gps_sensor}" />  <!-- [kg] -->
-        <origin xyz="0 0 0" rpy="0 0 0" />
-      </inertial>
-    </link>
-    <!-- GPS joint -->
-    <joint name="${namespace}/gps${gps_suffix}_joint" type="revolute">
-      <xacro:insert_block name="origin" />
-      <parent link="${parent_link}" />
-      <child link="${namespace}/gps${gps_suffix}_link" />
-      <limit upper="0" lower="0" effort="0" velocity="0" />
-    </joint>
-    <gazebo reference="${namespace}/gps${gps_suffix}_link">
-      <sensor type="gps" name="${namespace}_gps${gps_suffix}">
-        <pose>0 0 0 0 0 0</pose>
-        <visualize>0</visualize>
-        <always_on>1</always_on>
-        <update_rate>5</update_rate>
-        <gps>
-          <position_sensing>
-            <horizontal>
-              <noise type="gaussian">
-                <mean>0.0</mean>
-                <stddev>${horizontal_pos_std_dev}</stddev>
-                <bias_mean>0.0</bias_mean>
-                <bias_stddev>0.0</bias_stddev>
-              </noise>
-            </horizontal>
-            <vertical>
-              <noise type="gaussian">
-                <mean>0.0</mean>
-                <stddev>${vertical_pos_std_dev}</stddev>
-                <bias_mean>0.0</bias_mean>
-                <bias_stddev>0.0</bias_stddev>
-              </noise>
-            </vertical>
-          </position_sensing>
-          <velocity_sensing>
-            <horizontal>
-              <noise type="gaussian">
-                <mean>0.0</mean>
-                <stddev>${horizontal_vel_std_dev}</stddev>
-                <bias_mean>0.0</bias_mean>
-                <bias_stddev>0.0</bias_stddev>
-              </noise>
-            </horizontal>
-            <vertical>
-              <noise type="gaussian">
-                <mean>0.0</mean>
-                <stddev>${vertical_vel_std_dev}</stddev>
-                <bias_mean>0.0</bias_mean>
-                <bias_stddev>0.0</bias_stddev>
-              </noise>
-            </vertical>
-          </velocity_sensing>
-        </gps>
-        <plugin filename="librotors_gazebo_gps_plugin.so" name="rotors_gazebo_gps${gps_suffix}_plugin">
-          <robotNamespace>${namespace}</robotNamespace> <!-- (string, required): ros namespace in which the messages are published -->
-          <linkName>${namespace}/gps${gps_suffix}_link</linkName> <!-- (string, required): name of the body which holds the GPS sensor -->
-          <gpsTopic>${gps_topic}</gpsTopic> <!-- (string): name of the sensor output topic and prefix of service names (defaults to 'gps') -->
-          <groundSpeedTopic>${ground_speed_topic}</groundSpeedTopic> <!-- (string): name of the ground speed output topic (defaults to 'ground_speed') -->
-          <horPosStdDev>${horizontal_pos_std_dev}</horPosStdDev> <!-- standard deviation for horizontal position noise [m] -->
-          <verPosStdDev>${vertical_pos_std_dev}</verPosStdDev> <!-- standard deviation for vertical position noise [m] -->
-          <horVelStdDev>${horizontal_vel_std_dev}</horVelStdDev> <!-- standard deviation for horizontal speed noise [m/s] -->
-          <verVelStdDev>${vertical_vel_std_dev}</verVelStdDev> <!-- standard deviation for vertical speed noise [m/s] -->
-        </plugin>
-      </sensor>
-    </gazebo>
-  </xacro:macro>
-  <!-- Macro to add a magnetometer. -->
-  <xacro:macro name="magnetometer_plugin_macro"
-    params="namespace magnetometer_suffix parent_link magnetometer_topic
+        <!-- GPS link -->
+        <link name="${namespace}/gps${gps_suffix}_link">
+            <inertial>
+                <xacro:insert_block name="inertia"/>
+                <mass value="${mass_gps_sensor}"/>  <!-- [kg] -->
+                <origin xyz="0 0 0" rpy="0 0 0"/>
+            </inertial>
+        </link>
+        <!-- GPS joint -->
+        <joint name="${namespace}/gps${gps_suffix}_joint" type="revolute">
+            <xacro:insert_block name="origin"/>
+            <parent link="${parent_link}"/>
+            <child link="${namespace}/gps${gps_suffix}_link"/>
+            <limit upper="0" lower="0" effort="0" velocity="0"/>
+        </joint>
+        <gazebo reference="${namespace}/gps${gps_suffix}_link">
+            <sensor type="gps" name="${namespace}_gps${gps_suffix}">
+                <pose>0 0 0 0 0 0</pose>
+                <visualize>0</visualize>
+                <always_on>1</always_on>
+                <update_rate>5</update_rate>
+                <gps>
+                    <position_sensing>
+                        <horizontal>
+                            <noise type="gaussian">
+                                <mean>0.0</mean>
+                                <stddev>${horizontal_pos_std_dev}</stddev>
+                                <bias_mean>0.0</bias_mean>
+                                <bias_stddev>0.0</bias_stddev>
+                            </noise>
+                        </horizontal>
+                        <vertical>
+                            <noise type="gaussian">
+                                <mean>0.0</mean>
+                                <stddev>${vertical_pos_std_dev}</stddev>
+                                <bias_mean>0.0</bias_mean>
+                                <bias_stddev>0.0</bias_stddev>
+                            </noise>
+                        </vertical>
+                    </position_sensing>
+                    <velocity_sensing>
+                        <horizontal>
+                            <noise type="gaussian">
+                                <mean>0.0</mean>
+                                <stddev>${horizontal_vel_std_dev}</stddev>
+                                <bias_mean>0.0</bias_mean>
+                                <bias_stddev>0.0</bias_stddev>
+                            </noise>
+                        </horizontal>
+                        <vertical>
+                            <noise type="gaussian">
+                                <mean>0.0</mean>
+                                <stddev>${vertical_vel_std_dev}</stddev>
+                                <bias_mean>0.0</bias_mean>
+                                <bias_stddev>0.0</bias_stddev>
+                            </noise>
+                        </vertical>
+                    </velocity_sensing>
+                </gps>
+                <plugin filename="librotors_gazebo_gps_plugin.so" name="rotors_gazebo_gps${gps_suffix}_plugin">
+                    <!-- (string, required): ros namespace in which the messages are published -->
+                    <robotNamespace>${namespace}</robotNamespace>
+                    <!-- (string, required): name of the body which holds the GPS sensor -->
+                    <linkName>${namespace}/gps${gps_suffix}_link</linkName>
+                    <!-- (string): name of the sensor output topic and prefix of service names (defaults to 'gps') -->
+                    <gpsTopic>${gps_topic}</gpsTopic>
+                    <!-- (string): name of the ground speed output topic (defaults to 'ground_speed') -->
+                    <groundSpeedTopic>${ground_speed_topic}</groundSpeedTopic>
+                    <!-- standard deviation for horizontal position noise [m] -->
+                    <horPosStdDev>${horizontal_pos_std_dev}</horPosStdDev>
+                    <!-- standard deviation for vertical position noise [m] -->
+                    <verPosStdDev>${vertical_pos_std_dev}</verPosStdDev>
+                    <!-- standard deviation for horizontal speed noise [m/s] -->
+                    <horVelStdDev>${horizontal_vel_std_dev}</horVelStdDev>
+                    <!-- standard deviation for vertical speed noise [m/s] -->
+                    <verVelStdDev>${vertical_vel_std_dev}</verVelStdDev>
+                </plugin>
+            </sensor>
+        </gazebo>
+    </xacro:macro>
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