Commit message: Starting control

File: gyro_description/urdf/moto.xacro (robot description, xacro)
@@ -8,5 +8,5 @@
     <xacro:property name="width" value="1.2"/>
     <xacro:property name="length" value="2"/>
-    <xacro:property name="mass_base" value="1"/>
+    <xacro:property name="mass_base" value="10"/>
     <!-- Properties of wheels    -->
     <xacro:property name="radius" value="0.3"/>
@@ -20,5 +20,5 @@
     <xacro:property name="radius_gyro" value=".4"/>
     <xacro:property name="h_gyro" value=".1"/>
-    <xacro:property name="mass_gyro" value="0.5"/>
+    <xacro:property name="mass_gyro" value="1"/>
     <!-- Include Gazebo association -->
     <xacro:include filename="$(find gyro_description)/urdf/moto.gazebo"/>
@@ -200,5 +200,5 @@
         <child link="axel_gyro_link"/>
         <axis xyz="0.0 1 0.0"/>
-        <limit lower="-${PI/2}" upper="${PI/2}" effort="20.0" velocity="10.0"/>
+        <limit lower="-${PI/2}" upper="${PI/2}" effort="20.0" velocity="100.0"/>
     </joint>
     <link name="axel_gyro_link">

Commit message: Feedback state space control

File: gyro_description/urdf/moto.xacro (robot description, xacro)
@@ -20,5 +20,5 @@
     <xacro:property name="radius_gyro" value=".4"/>
     <xacro:property name="h_gyro" value=".1"/>
-    <xacro:property name="mass_gyro" value="1"/>
+    <xacro:property name="mass_gyro" value="3"/>
     <!-- Include Gazebo association -->
     <xacro:include filename="$(find gyro_description)/urdf/moto.gazebo"/>
@@ -279,7 +279,7 @@
         <child link="gyro_link"/>
         <axis xyz="0.0 0.0 1"/>
-        <limit effort="50.0" velocity="200.0"/>
+        <limit effort="100.0" velocity="500.0"/>
         <safety_controller k_velocity="100.0"/>
-        <dynamics damping="0.1" friction="0.01"/>
+        <dynamics damping="0.1" friction="0.0"/>
     </joint>
     <link name="gyro_link">

Commit message: beggining Kalman

File: gyro_description/urdf/moto.xacro (robot description, xacro)
@@ -11,5 +11,5 @@
     <!-- Properties of wheels    -->
     <xacro:property name="radius" value="0.3"/>
-    <xacro:property name="h" value=".01"/>
+    <xacro:property name="h" value=".05"/>
     <xacro:property name="mass_wheel" value="0.2"/>
     <!-- Properties from gyro support -->
@@ -93,14 +93,14 @@
             <origin xyz="0.0 0.0 0.0" rpy="${PI/2} 0.0 0.0"/>
             <geometry>
-<!--                <sphere radius="${radius}"/>-->
-                <cylinder radius="${radius}" length="${h}"/>
-                <!-- <mesh filename="${mesh_base}" scale="1.0"/> -->
-            </geometry>
-        </visual>
-        <collision>
-            <origin xyz="0.0 0.0 0.0" rpy="${PI/2} 0.0 0.0"/>
-            <geometry>
-<!--                <sphere radius="${radius}"/>-->
-                <cylinder radius="${radius}" length="${h}"/>
+                <!--  <cylinder radius="${radius}" length="${h}"/>-->
+                <!-- <mesh filename="${mesh_base}" scale="1.0"/> -->
+                <sphere radius="${radius}"/>
+            </geometry>
+        </visual>
+        <collision>
+            <origin xyz="0.0 0.0 0.0" rpy="${PI/2} 0.0 0.0"/>
+            <geometry>
+                <!-- <cylinder radius="${radius}" length="${h}"/>-->
+                <sphere radius="${radius}"/>
                 <!-- <origin xyz="0.0 0.0 0.0" rpy="0.0 0.0 0.0"/> -->
             </geometry>
@@ -118,13 +118,15 @@
             <origin xyz="0.0 0.0 0.0" rpy="${PI/2} 0.0 0.0"/>
             <geometry>
-                <cylinder radius="${radius}" length="${h}"/>
-                <!-- <mesh filename="${mesh_base}" scale="1.0"/> -->
-            </geometry>
-        </visual>
-        <collision>
-            <origin xyz="0.0 0.0 0.0" rpy="${PI/2} 0.0 0.0"/>
-            <geometry>
-                <cylinder radius="${radius}" length="${h}"/>
-                <!-- <origin xyz="0.0 0.0 0.0" rpy="0.0 0.0 0.0"/> -->
+                <!-- <cylinder radius="${radius}" length="${h}"/>-->
+                <!-- <mesh filename="${mesh_base}" scale="1.0"/> -->
+                <sphere radius="${radius}"/>
+            </geometry>
+        </visual>
+        <collision>
+            <origin xyz="0.0 0.0 0.0" rpy="${PI/2} 0.0 0.0"/>
+            <geometry>
+                <!-- <cylinder radius="${radius}" length="${h}"/>-->
+                <!-- <origin xyz="0.0 0.0 0.0" rpy="0.0 0.0 0.0"/> -->
+                <sphere radius="${radius}"/>
             </geometry>
         </collision>

Commit message: Updating code

File: gyro_description/urdf/moto.xacro (robot description, xacro)
@@ -5,24 +5,41 @@
     <xacro:property name="PI" value="3.1415926535897931"/>
     <!-- Properties of base -->
+    <xacro:property name="height" value=".2"/>
+    <xacro:property name="width" value="1.2"/>
+    <xacro:property name="length" value="2"/>
+    <xacro:property name="mass_base" value="10"/>
+    <!-- Properties of wheels    -->
+    <xacro:property name="radius" value="0.3"/>
+    <xacro:property name="h" value=".05"/>
+    <xacro:property name="mass_wheel" value="0.2"/>
+    <!-- Properties from gyro support -->
+    <xacro:property name="mass_support" value="1"/>
+    <xacro:property name="h_support" value="0.5"/>
+    <xacro:property name="w_support" value="0.1"/>
+    <!-- Propertis of a gyroscope -->
+    <xacro:property name="radius_gyro" value=".4"/>
+    <xacro:property name="h_gyro" value=".1"/>
+    <xacro:property name="mass_gyro" value="3"/>
+<!--    &lt;!&ndash; Properties of base &ndash;&gt;
     <xacro:property name="height" value="2"/>
     <xacro:property name="width" value="12"/>
     <xacro:property name="length" value="20"/>
     <xacro:property name="mass_base" value="100"/>
-    <!-- Properties of wheels    -->
+    &lt;!&ndash; Properties of wheels    &ndash;&gt;
     <xacro:property name="radius" value="3"/>
     <xacro:property name="h" value=".5"/>
     <xacro:property name="mass_wheel" value="2"/>
-    <!-- Properties from gyro support -->
+    &lt;!&ndash; Properties from gyro support &ndash;&gt;
     <xacro:property name="mass_support" value="10"/>
     <xacro:property name="h_support" value="5"/>
     <xacro:property name="w_support" value="1"/>
-    <xacro:property name="effort_support" value="20000"/>
-    <xacro:property name="velocity_support" value="1000"/>
-    <!-- Propertis of a gyroscope -->
+    &lt;!&ndash; Propertis of a gyroscope &ndash;&gt;
     <xacro:property name="radius_gyro" value="4"/>
     <xacro:property name="h_gyro" value="1"/>
-    <xacro:property name="mass_gyro" value="30"/>
-    <xacro:property name="effort_gyro" value="2000"/>
-    <xacro:property name="velocity_gyro" value="1000"/>
+    <xacro:property name="mass_gyro" value="30"/>-->
+    <xacro:property name="effort_support" value="200"/>
+    <xacro:property name="velocity_support" value="100"/>
+    <xacro:property name="effort_gyro" value="200"/>
+    <xacro:property name="velocity_gyro" value="200"/>
     <xacro:property name="k_velocity_gyro" value="100"/>
     <xacro:property name="damp_gyro" value="0.1"/>
